Commit message: Added use_gazebo condition

File: config/fr3.ros2_control.xacro (robot description, xacro)
@@ -1,10 +1,14 @@
 <?xml version="1.0"?>
 <robot xmlns:xacro="http://www.ros.org/wiki/xacro">
-    <xacro:macro name="fr3_ros2_control" params="name initial_positions_file">
+    <xacro:macro name="fr3_ros2_control" params="name initial_positions_file use_gazebo">
         <xacro:property name="initial_positions" value="${load_yaml(initial_positions_file)['initial_positions']}"/>
         <ros2_control name="${name}" type="system">
             <hardware>
-                <!-- By default, set up controllers for simulation. This won't work on real hardware -->
+              <xacro:if value="${use_gazebo}">
+                <plugin>gz_ros2_control/GazeboSimSystem</plugin>
+              </xacro:if>
+              <xacro:unless value="${use_gazebo}">
                 <plugin>mock_components/GenericSystem</plugin>
+              </xacro:unless>
             </hardware>
             <joint name="fr3_joint_linear">

File: config/fr3.urdf.xacro (robot description, xacro)
@@ -2,8 +2,23 @@
 <robot xmlns:xacro="http://www.ros.org/wiki/xacro" name="fr3">
     <xacro:arg name="initial_positions_file" default="initial_positions.yaml" />
+    <xacro:arg name="use_gazebo" default="false"/>
     <!-- Import fr3 urdf file -->
     <xacro:include filename="$(find fr3_description)/urdf/fr3.urdf" />
     <!-- Import control_xacro -->
     <xacro:include filename="fr3.ros2_control.xacro" />
-    <xacro:fr3_ros2_control name="FakeSystem" initial_positions_file="$(arg initial_positions_file)"/>
+    <!-- Import ros2_control tag -->
+    <xacro:fr3_ros2_control
+        name="FrankaSystem"
+        initial_positions_file="$(arg initial_positions_file)"
+        use_gazebo="$(arg use_gazebo)"/>
+    <!-- Gazebo plugin, if using gazebo -->
+    <xacro:if value="$(arg use_gazebo)">
+        <gazebo>
+            <plugin filename="libgz_ros2_control-system.so" name="gz_ros2_control::GazeboSystemInterface">
+                <robot_param>robot_description</robot_param>
+                <robot_param_node>robot_state_publisher</robot_param_node>
+                <parameters>package://fr3_moveit_config/config/ros2_controllers.yaml</parameters>
+            </plugin>
+        </gazebo>
+    </xacro:if>
 </robot>
