Commit message: Add world link to stabilize joint vibrating

File: config/fr3.urdf.xacro (robot description, xacro)
@@ -3,4 +3,10 @@
     <xacro:arg name="initial_positions_file" default="initial_positions.yaml" />
     <xacro:arg name="use_gazebo" default="false"/>
+    <link name="world"/>
+    <joint name="world_to_stationary" type="fixed">
+        <parent link="world"/>
+        <child link="fr3_link_stationary"/>
+        <origin xyz="0 0 0" rpy="0 0 0"/>
+    </joint>
     <!-- Import fr3 urdf file -->
     <xacro:include filename="$(find fr3_description)/urdf/fr3.urdf" />
@@ -15,8 +21,8 @@
     <xacro:if value="$(arg use_gazebo)">
         <gazebo>
-            <plugin filename="libgz_ros2_control-system.so" name="gz_ros2_control::GazeboSystemInterface">
+            <plugin filename="libgz_ros2_control-system.so" name="gz_ros2_control::GazeboSimROS2ControlPlugin">
                 <robot_param>robot_description</robot_param>
                 <robot_param_node>robot_state_publisher</robot_param_node>
-                <parameters>package://fr3_moveit_config/config/ros2_controllers.yaml</parameters>
+                <parameters>$(find fr3_moveit_config)/config/ros2_controllers.yaml</parameters>
             </plugin>
         </gazebo>
